File: NEC-DE10.kicad_sch (KiCad schematic)
At the start: 12 parts, among them U3 74ALVC164245, U4 74ALVC164245, U5 74ALVC164245

Commit message: Added V35 board
Parts:
- removed C1, C2, C3, C4, C5, C6, C7: 100nF, Capacitor_SMD:C_0603_1608Metric, symbol Device:C_Small
- removed U1: ~, Package_DIP:DIP-40_W15.24mm_Socket, symbol NEC-DE10:V30
- removed U2: ~, NEC-DE10:MODULE_P0496, symbol NEC-DE10:P0496
- removed U3, U4, U5: 74ALVC164245, Package_SO:TSSOP-48_6.1x12.5mm_P0.5mm, symbol 74xx:74ALVC164245
Other:
- added sheet V35 (v35.kicad_sch)
- sheet V30: file untitled.kicad_sch -> v30.kicad_sch
